File: Hardware/Production/Thing_Plus_MGM240P-Panel.brd (EAGLE design)
At the start: 89.7 x 72.6 mm, 519 parts, among them J1 THING_PLUS_LOGICAL, J10 QWIIC_RIGHT_ANGLE, J11 MICRO-SDFRICTION, J13 THING_PLUS_LOGICAL, J14 USB Female Type C Connector, J16 QWIIC_RIGHT_ANGLE, J17 MICRO-SDFRICTION, J2 USB Female Type C Connector, J3 QWIIC_RIGHT_ANGLE, J5 MICRO-SDFRICTION, J6 THING_PLUS_LOGICAL, J8 USB Female Type C Connector, Q1 20V/4.2A/52mΩ/1.4W, Q2 20V/4.2A/52mΩ/1.4W, Q3 20V/4.2A/52mΩ/1.4W, U1 MGM240P, U10 MCP73831, U11 MAX17048, U12 EFM32GG12B410F1024GL120, U13 M24C02-FMC6TG, U14 MX25R8035FZUIL0, U15 MGM240P, U16 XC6222B331MR-G, U17 MCP73831, U18 MAX17048, U19 EFM32GG12B410F1024GL120, U2 XC6222B331MR-G, U20 M24C02-FMC6TG, U21 MX25R8035FZUIL0, U3 EFM32GG12B410F1024GL120, U4 MCP73831, U5 MAX17048, U6 M24C02-FMC6TG, U7 MX25R8035FZUIL0, U8 MGM240P, U9 XC6222B331MR-G, Y1 CRYSTAL-48MHZ, Y2 CRYSTAL-48MHZ, Y3 CRYSTAL-48MHZ

Commit message: Update proto production files for v02
Parts:
- R15, R32, R50: value 4.7k -> 2.2k
- U$112, U$190: device output:#_A7#0 -> output:#_C5#0
- U$113, U$191: device output:#_C5#0 -> output:#_C4#0
- U$114, U$192: device output:#_C4#0 -> output:#C7_#0
- U$115, U$193: device output:#C7_#0 -> output:#A5_#0
- U$116, U$194: device output:#A5_#0 -> output:#A6_#0
- U$117, U$195: device output:#A6_#0 -> output:#C6_#0
- U$118, U$196: device output:#C6_#0 -> output:#C3_#0
- U$119, U$197: device output:#C3_#0 -> output:#C2_#0
- U$120, U$198: device output:#C2_#0 -> output:#C1_#0
- U$121, U$199: device output:#C1_#0 -> output:#C0_#0
- U$122, U$200: device output:#C0_#0 -> output:#D0_#0
- U$123, U$201: device output:#D0_#0 -> output:#D1_#0
- U$124, U$202: device output:#D1_#0 -> output:#_C1#0
- U$125, U$203: device output:#_C1#0 -> output:#_C0#0
- U$126, U$204: device output:#_C0#0 -> output:#_D0#0
- U$127, U$205: device output:#_D0#0 -> output:#_D1#0
- U$128, U$206: device output:#_D1#0 -> output:#_D2#0
- U$129, U$207: device output:#_D2#0 -> output:#_D3#0
- U$130, U$208: device output:#_D3#0 -> output:#C4_#0
- U$131, U$209: device output:#C4_#0 -> output:#C5_#0
- U$132, U$210: device output:#C5_#0 -> output:#A0_#0
- U$133, U$211: device output:#A7_#0 -> output:#B0_#0
- U$134, U$212: device output:#A0_#0 -> output:#B2_#0
- U$135, U$213: device output:#B0_#0 -> output:#B1_#0
- U$136, U$214: device output:#B2_#0 -> output:#SDA#B4_#0
- U$137, U$215: device output:#B1_#0 -> output:#SCL#B3_#0
- U$138, U$216: device output:#SDA#B4_#0 -> output:#_A5#TX#0
- U$139, U$217: device output:#SCL#B3_#0 -> output:#_A6#RX#0
- U$140, U$218: device output:#_A5#TX#0 -> output:#_C6#POCI#0
- U$141, U$219: device output:#_A6#RX#0 -> output:#_C3#PICO#0
- U$142, U$220: device output:#_C6#POCI#0 -> output:#_C2#SCK#0
- U$143, U$221: device output:#_C3#PICO#0 -> output:MINI_SIMPLICITY0
- U$144, U$222: device output:#_C2#SCK#0 -> output:A80
- U$145, U$223: device output:MINI_SIMPLICITY0 -> output:MEAS81
- U$146, U$224: device output:A80 -> SparkFun-Aesthetics:ORDERING_INSTRUCTIONS
- U$147, U$225: device output:MEAS81 -> SparkFun-Aesthetics:FOUR_LAYER_WARNING
- U$148, U$226: device SparkFun-Aesthetics:ORDERING_INSTRUCTIONS -> output:#0#5A#0
- U$149, U$227: device SparkFun-Aesthetics:FOUR_LAYER_WARNING -> output:#0#1A#0
- U$150, U$228: device output:#0#5A#0 -> output:#D2_#0
- U$151, U$229: device output:#0#1A#0 -> output:#D3_#0
- U$152, U$230: device output:#D2_#0 -> output:DBG0
- U$153, U$231: device output:#D3_#0 -> output:#_C7#FREE#0
- U$154, U$232: device output:DBG0 -> output:#LP#0
- U$155, U$233: device output:#_C7#FREE#0 -> output:#_A4#0
- U$156, U$234: device output:#LP#0 -> output:#A4_#0
- U$50: device output:#A7_#0 -> output:#A4_#0
- U$8: device output:#_A7#0 -> output:#_A4#0
- moved U$148 43.3 mm to (37.7, 14.6), flipped to the bottom, turned to 90 degrees
- moved U$226 43.3 mm to (61.1, 14.6), flipped to the bottom, turned to 90 degrees
- moved U$149 34.0 mm to (39.5, 14.6), flipped to the bottom, turned to 90 degrees
- moved U$227 34.0 mm to (62.9, 14.6), flipped to the bottom, turned to 90 degrees
- moved U$147 33.1 mm to (62.7, 39.4)
- moved U$225 33.1 mm to (86.1, 39.4)
- moved U$146 32.6 mm to (61.5, 50.8), turned to 0 degrees
- moved U$224 32.6 mm to (84.8, 50.8), turned to 0 degrees
- moved U$145 31.1 mm to (43.7, 12.3)
- moved U$223 31.1 mm to (67.1, 12.3)
- moved U$153 27.9 mm to (45.0, 52.1), flipped to the bottom
- moved U$231 27.9 mm to (68.3, 52.1), flipped to the bottom
- moved U$114 27.0 mm to (45.0, 52.1)
- moved U$192 27.0 mm to (68.3, 52.1)
- moved U$155 25.4 mm to (24.6, 36.8), flipped to the top
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Connections:
- removed net PA06: J17.2, U15.11
- removed net PA07: J1.7, U1.16
- removed net PA08: J13.7, U15.16
- new net !SD_CS!/PA01: J11.2, U8.16
- new net !SD_CS!/PA02: J17.2, U15.16
- new net !SD_CS!/PA07: J5.2, U1.16
- net DBG_RX: now also TP13.1, U3.A1; no longer TP14.1, U3.A2
- net DBG_RX1: now also TP27.1, U12.A1; no longer TP28.1, U12.A2
- net DBG_RX2: now also TP41.1, U19.A1; no longer TP42.1, U19.A2
- net DBG_TX: now also TP14.1, U3.A2; no longer TP13.1, U3.A1
- net DBG_TX1: now also TP28.1, U12.A2; no longer TP27.1, U12.A1
- net DBG_TX2: now also TP42.1, U19.A2; no longer TP41.1, U19.A1
- net PA02: now also J6.7; no longer J11.2
- net PA03: now also J13.6, U15.7; no longer J6.7, U8.16
- net PA04: now also J1.7; no longer J5.2
- net PA05: now also J13.7, U15.11; no longer J13.6, U15.7
Routing:
- net PA06: track 33.7 -> 0.00 mm, vias 3 -> 0
- net !SD_CS!/PA02: track 0.00 -> 31.7 mm, vias 0 -> 3
- net !SD_CS!/PA07: track 0.00 -> 31.7 mm, vias 0 -> 3
- net !SD_CS!/PA01: track 0.00 -> 31.7 mm, vias 0 -> 3
- net PA04: track 33.7 -> 14.0 mm, vias 3 -> 0
- net PA02: track 33.7 -> 14.0 mm, vias 3 -> 0
- net PA07: track 12.3 -> 0.00 mm
- net PA08: track 12.3 -> 0.00 mm
- net GND: track 113.9 -> 119.9 mm, vias 112 -> 115
- net GND1: track 113.9 -> 119.9 mm, vias 112 -> 115
- net GND2: track 113.9 -> 119.9 mm, vias 112 -> 115
- net PA03: track 12.3 -> 14.7 mm
- net DBG_TX1: track 4.16 -> 2.69 mm
- net DBG_RX1: track 2.69 -> 4.16 mm
- net DBG_TX2: track 4.16 -> 2.69 mm
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Other:
- board text added: "v02"
- board text removed: "v01"
